File: kiCad/ff-led-panel/ff-led-panel.kicad_pcb (KiCad board)
At the start: 2 copper layers, 23 x 76 mm, 10 parts, among them J2 Conn_01x02_Socket, J5 RJ14, U1 XIAO-ESP32-C3-DIP, U2 MAX3232, U3 R-785.0-0.5

Commit message: Create gerbe files for pcb
Parts:
- removed J2: Conn_01x02_Socket, Connector_JST:JST_EH_S2B-EH_1x02_P2.50mm_Horizontal
- removed J5: RJ14, Connector_RJ:RJ14_Connfly_DS1133-S4_Horizontal
- added 12V: DC050-T, DC_PowerJack:DC-IN_DC050-T, F.Cu at (135.7, 135.9)
- added C6: 100nF, PCM_JLCPCB:C_0402, F.Cu at (135.5, 95.0)
- added C7: 100nF, PCM_JLCPCB:C_0402, F.Cu at (139.5, 85.0)
- added D1: 1N5819WS, PCM_JLCPCB:D_SOD-323, F.Cu at (141.2, 118.0)
- added RS232: PCB-6P4C-90_C189746, RJ11:RJ11-TH_PCB-6P4C-90_C189746, F.Cu at (135.2, 78.1)
- C1: value 1uF -> 10uF; footprint Capacitor_SMD:C_0201_0603Metric -> PCM_JLCPCB:C_1206
- C2: value 1uF -> 22uF; footprint Capacitor_SMD:C_0201_0603Metric -> PCM_JLCPCB:C_1206
- C3, C4: value 1uF -> 100nF; footprint Capacitor_SMD:C_0201_0603Metric -> PCM_JLCPCB:C_0402
- C5: value C -> 100nF; footprint Capacitor_SMD:C_0201_0603Metric -> PCM_JLCPCB:C_0402
- U1: footprint ff-led-panel:XIAO-ESP32C3-DIP -> esp32:XIAO-ESP32C3-DIP
- U3: value R-785.0-0.5 -> AMS1117; footprint Converter_DCDC:Converter_DCDC_RECOM_R-78E-0.5_THT -> PCM_JLCPCB:SOT-223_L6.5-W3.5-P2.30-LS7.0-BR
- moved C2 29.5 mm to (136.0, 118.0), turned to 180 degrees
- moved C1 27.1 mm to (130.2, 118.0), turned to 180 degrees
- moved C5 9.73 mm to (139.5, 88.5), turned to 90 degrees
- moved C3 9.00 mm to (128.5, 92.0), turned to 180 degrees
- moved C4 5.81 mm to (139.5, 92.0), turned to 90 degrees
- moved U3 2.94 mm to (135.0, 125.0), turned to 90 degrees
- moved U1 2.09 mm to (134.6, 105.6)
Connections:
- net Net-(U1-GPIO2/A0/D0) renamed /UART RX
- net Net-(U1-GPIO3/A1/D1) renamed /UART TX
- C1 pad 1: Net-(U2-C1+) -> /12V
- C1 pad 2: Net-(U2-C1-) -> GND
- C2 pad 1: Net-(U2-C2+) -> /5V
- C2 pad 2: Net-(U2-C2-) -> GND
- C3 pad 1: Net-(U2-VS+) -> /3.3V
- C4 pad 1: GND -> Net-(U2-C1+)
- C4 pad 2: Net-(U2-VS-) -> Net-(U2-C1-)
- C5 pad 1: Net-(U1-VCC_3V3) -> Net-(U2-C2+)
- C5 pad 2: GND -> Net-(U2-C2-)
- U1 pad 12: Net-(U1-VCC_3V3) -> /3.3V
- U1 pad 14: Net-(U1-VBUS) -> /5VD
- U2 pad 13: Net-(U2-R1IN) -> /RS232 RX
- U2 pad 14: Net-(U2-T1OUT) -> /RS232 TX
- U2 pad 16: Net-(U1-VCC_3V3) -> /3.3V
- U3 pad 1: Net-(J2-Pin_2) -> GND
- U3 pad 2: GND -> /5V
- U3 pad 3: Net-(U1-VBUS) -> /12V
Routing:
- net /3.3V: track 0.00 -> 26.6 mm
- net /12V: track 0.00 -> 26.2 mm
- net Net-(U1-VCC_3V3): track 25.5 -> 0.00 mm
- net /RS232 TX: track 0.00 -> 17.6 mm
- net /5V: track 0.00 -> 16.1 mm
- net Net-(U2-T1OUT): track 15.7 -> 0.00 mm
- net Net-(U1-VBUS): track 13.8 -> 0.00 mm
- net Net-(U2-R1IN): track 13.2 -> 0.00 mm
- net /RS232 RX: track 0.00 -> 13.0 mm
- net Net-(J2-Pin_2): track 10.4 -> 0.00 mm
- net /5VD: track 0.00 -> 4.94 mm
- net /UART RX: track 19.9 -> 15.9 mm
- net /UART TX: track 16.9 -> 17.1 mm, vias 0 -> 1
