File: kiCad/ff-led-panel/ff-led-panel.kicad_sch (KiCad schematic)
At the start: 10 parts, among them J2 Conn_01x02_Socket, J5 RJ14, U1 XIAO-ESP32-C3-DIP, U2 MAX3232, U3 R-785.0-0.5

Commit message: Create gerbe files for pcb
Parts:
- removed C1, C2, C3, C4: 1uF, Capacitor_SMD:C_0201_0603Metric, symbol Device:C
- removed C5: C, Capacitor_SMD:C_0201_0603Metric, symbol Device:C
- removed J2: Conn_01x02_Socket, Connector_JST:JST_EH_S2B-EH_1x02_P2.50mm_Horizontal, symbol Connector:Conn_01x02_Socket
- removed J5: RJ14, Connector_RJ:RJ14_Connfly_DS1133-S4_Horizontal, symbol Connector:RJ14
- removed U3: R-785.0-0.5, Converter_DCDC:Converter_DCDC_RECOM_R-78E-0.5_THT, symbol Regulator_Switching:R-785.0-0.5
- added C1: 10uF, PCM_JLCPCB:C_1206, symbol PCM_JLCPCB-Capacitors:1206,10uF
- added C2: 22uF, PCM_JLCPCB:C_1206, symbol PCM_JLCPCB-Capacitors:1206,22uF,(2)
- added C3, C4, C5, C6, C7: 100nF, PCM_JLCPCB:C_0402, symbol PCM_JLCPCB-Capacitors:0402,100nF
- added D1: 1N5819WS, PCM_JLCPCB:D_SOD-323, symbol PCM_JLCPCB-Diodes:Schottky,1N5819WS
- added RJ11: PCB-6P4C-90_C189746, RJ11:RJ11-TH_PCB-6P4C-90_C189746, symbol RJ11:PCB-6P4C-90_C189746
- added U3: AMS1117, PCM_JLCPCB:SOT-223_L6.5-W3.5-P2.30-LS7.0-BR, symbol PCM_JLCPCB-Power:LDO, 5V, 1A
- U1: footprint ff-led-panel:XIAO-ESP32C3-DIP -> esp32:XIAO-ESP32C3-DIP
Connections:
- net GND: now also C1.2, C2.2, C3.2, C6.2, C7.2, RJ11.4, U3.1 (GND)
- net 5VD: now reaches U1.14 (VBUS)
- net 5VD: now also D1.1
- net 3.3V: now reaches U1.12 (VCC_3V3), U2.16 (VCC)
- net 3.3V: now also C3.1
- net at U2.4 (C2+): now also C5.1
- net at U2.5 (C2-): now also C5.2
- net RS232 TX: now reaches U2.14 (T1OUT)
- net RS232 TX: now also RJ11.1
- net RS232 RX: now reaches U2.13 (R1IN)
- net RS232 RX: now also RJ11.2
- net at U2.1 (C1+): now also C4.1
- net at U2.3 (C1-): now also C4.2
- net UART RX: now reaches U1.1 (GPIO2/A0/D0), U2.12 (R1OUT)
- net UART TX: now reaches U1.2 (GPIO3/A1/D1), U2.11 (T1IN)
- net at U2.6 (VS-): now also C7.1
- net at U2.2 (VS+): now also C6.1
- new net 12V: C1.1, U3.3 (VIN)
- new net 5V: C2.1, D1.2, U3.2 (VOUT), U3.4 (VOUT)
- no-connect marks 13 -> 14
